File: Kicad/Temp_RH/Remote_Temp_RH/Temp_RH.sch (KiCad schematic (older format))
At the start: 13 parts, among them J1 DHT 11, J2 Arduino, J3 DHT 22, J4 SHT 75, J5 SHT 31

Commit message: Kicad Current project update Kicad TH project update
Parts:
- removed D1, D2: LED, LEDs:LED_D1.8mm_W3.3mm_H2.4mm, symbol LED
- removed J2: Arduino, Connectors_Terminal_Blocks:TerminalBlock_Pheonix_MPT-2.54mm_10pol, symbol Screw_Terminal_1x10
- removed J4: SHT 75, Pin_Headers:Pin_Header_Straight_1x04_Pitch1.27mm, symbol CONN_01X04
- removed R5: 1k, Resistors_THT:R_Axial_DIN0204_L3.6mm_D1.6mm_P5.08mm_Horizontal, symbol R
- added C2: 1u, Capacitors_THT:CP_Radial_D4.0mm_P1.50mm, symbol CP
- added J2: DHT 22, Pin_Headers:Pin_Header_Straight_1x04_Pitch1.27mm, symbol CONN_01X04
- added J4: Screw_Terminal_1x12, Connectors_Terminal_Blocks:TerminalBlock_Pheonix_MPT-2.54mm_12pol, symbol Screw_Terminal_1x12
- added J7: NTC, Pin_Headers:Pin_Header_Straight_1x02_Pitch1.27mm, symbol CONN_01X02
- added J8: MLX, Pin_Headers:Pin_Header_Straight_1x04_Pitch1.27mm, symbol CONN_01X04
- J3: value DHT 22 -> SHT 75
- R4: value 1k -> 10k
- renumbered C1 to Decouplador1
Connections:
- net labels added: Clock75, Data11, Data22, Data75, DataNTC, SCL31, SDA31, SLC31
- net labels removed: DataSHT75, Data_DHT11, Data_DHT22, Ground´, LedOut, LedPower, Reset, SKC_SHT75
- wire segments 64 -> 86
Other:
- moved on the sheet: Decouplador1, J1, R1, R2, R3, R4

Commit message: Revision V2.0! New version of remote aquisition system for Temperature and humidity.
Parts:
- removed J4: Screw_Terminal_1x12, Connectors_Terminal_Blocks:TerminalBlock_Pheonix_MPT-2.54mm_12pol, symbol Screw_Terminal_1x12
- added J10, J11, J4: CONN_01X02, Pin_Headers:Pin_Header_Straight_1x02_Pitch2.54mm, symbol CONN_01X02
- added J12, J6, J9: CONN_01X01, Pin_Headers:Pin_Header_Straight_1x01_Pitch2.54mm, symbol CONN_01X01
- C2, Decouplador1: footprint Capacitors_THT:CP_Radial_D4.0mm_P1.50mm -> Capacitors_THT:CP_Radial_D5.0mm_P2.50mm
- J1, J2, J3, J8: footprint Pin_Headers:Pin_Header_Straight_1x04_Pitch1.27mm -> Pin_Headers:Pin_Header_Straight_1x04_Pitch2.54mm
- J5: footprint Pin_Headers:Pin_Header_Straight_1x07_Pitch1.27mm -> Pin_Headers:Pin_Header_Straight_1x07_Pitch2.54mm
- J7: footprint Pin_Headers:Pin_Header_Straight_1x02_Pitch1.27mm -> Pin_Headers:Pin_Header_Straight_1x02_Pitch2.54mm
Connections:
- net labels added: SLC
- net labels removed: SCL31, SDA31, SLC31
- wire segments 86 -> 84
- no-connect marks 5 -> 4
